File: 2019-Pi-Power.kicad_pcb (KiCad board)
At the start: 2 copper layers, 65 x 56 mm, 132 parts, among them J1 Barrel_Jack_Switch, J2 USB_A, J3 USB_A, J4 Conn_02x04_Odd_Even, J5 Conn_01x04, J6 Conn_01x04, J7 Conn_01x04, J8 Conn_02x02_Odd_Even, P1 Conn_02x20_Odd_Even, U1 MP1584

Commit message: Silkscreen adjustments
Other:
- board text added: "5V"
Changed lines of the file:
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@@
   (general
     (thickness 1.6)
-    (drawings 62)
+    (drawings 63)
     (tracks 117)
     (zones 0)
@@
     (descr "Through hole straight pin header, 1x04, 2.54mm pitch, single row")
     (tags "Through hole pin header THT 1x04 2.54mm single row")
-    (fp_text reference J7 (at 0 -2.33 90) (layer F.SilkS)
+    (fp_text reference J7 (at 0.4445 -2.6035 180) (layer F.SilkS)
       (effects (font (size 1 1) (thickness 0.15)))
     )
@@
     (descr "Through hole straight pin header, 2x02, 2.54mm pitch, double rows")
     (tags "Through hole pin header THT 2x02 2.54mm double row")
-    (fp_text reference J8 (at -0.0635 -2.3495 90) (layer F.SilkS)
+    (fp_text reference J8 (at 2.667 -2.159 90) (layer F.SilkS)
       (effects (font (size 1 1) (thickness 0.15)))
     )
@@
       (xy 0.376964 -2.709982)) (layer F.SilkS) (width 0.01))
   )
-  (gr_text I2C (at 221.463 102.4385) (layer F.SilkS)
+  (gr_text 5V (at 252.8955 142.1895) (layer F.SilkS)
+    (effects (font (size 1 1) (thickness 0.15)))
+  )
+  (gr_text I2C (at 208.509 103.5815) (layer F.SilkS)
     (effects (font (size 1 1) (thickness 0.2)))
   )
